File: Kicad/Aforino.sch (KiCad schematic (older format))
At the start: 4 parts, among them U1 ESP-13-WROOM-02

Commit message: Under Contruction: Kicad
Parts:
- removed U1: ESP-13-WROOM-02, ESP8266:ESP-13-WROOM-02, symbol ESP-13-WROOM-02
- added J3: Conn_01x04_Female, symbol Conn_01x04_Female
- added SW1, SW2: SW_Push, Button_Switch_THT:SW_PUSH_6mm_h5mm, symbol SW_Push
- added U1: ESP-Breatout-16Pin, myLib:ESP-Breakout-16PIN, symbol ESP-Breatout-16Pin
Connections:
- net labels added: +3.3V, FIRM_SW, GND, IR_IN, IR_OUT, SDA, SDL
- wire segments 0 -> 37
- no-connect marks 0 -> 6
Other:
- moved on the sheet: Conn2

Commit message: Under Contruction: Kicad Pcbnew, Track and Vias
Parts:
- removed J3: Conn_01x04_Female, symbol Conn_01x04_Female
- removed uP1: ARDUPROMINI, ArduProMiniTKB:ArduProMini, symbol ARDUPROMINI
- added J1, J2: Conn_01x04_Female, Connector_PinHeader_2.54mm:PinHeader_1x04_P2.54mm_Vertical, symbol Conn_01x04_Female
- added SH1: ARDUINO_MINI_PRO, SHIELD_ARDUINO:ARDUINO_MINI_PRO_V10, symbol ARDUINO_MINI_PRO
- SW1, SW2: footprint Button_Switch_THT:SW_PUSH_6mm_h5mm -> Buttons_Switches_THT:SW_PUSH_6mm_h5mm
Connections:
- net labels added: SCL
- net labels removed: SDL
- wire segments 37 -> 44
- no-connect marks 6 -> 33
Other:
- moved on the sheet: Conn1, Conn2, SW1, SW2, U1

Commit message: Kidcat first testing board
Parts:
- added LM2596-1: myConn_LM2596_Male, myLib:myConn_LM2596_Male, symbol myConn_LM2596_Male
- SW1, SW2: footprint Buttons_Switches_THT:SW_PUSH_6mm_h5mm -> Buttons_Switches_THT:SW_PUSH_6mm
Connections:
- wire segments 44 -> 43
Other:
- moved on the sheet: J2

Commit message: Kicad: ESP8266 Breakout Shield Good! Jumpers to Upload firmware! Best component order!
Parts:
- removed J2: Conn_01x04_Female, Connector_PinHeader_2.54mm:PinHeader_1x04_P2.54mm_Vertical, symbol Conn_01x04_Female
- removed SW1, SW2: SW_Push, Buttons_Switches_THT:SW_PUSH_6mm, symbol SW_Push
- added P1, P2: CONN_01X02, Pin_Headers:Pin_Header_Straight_1x02, symbol CONN_01X02
- Conn1, Conn2: footprint myLib:myConn3x1 -> Escolabs:MyConn3x1
- J1: symbol Conn_01x04_Female -> Conn_01x04_Female-RESCUE-Aforino
- U1: footprint myLib:ESP-Breakout-16PIN -> Escolabs:ESP8266-Breakout_Board-16Pin
Connections:
- wire segments 43 -> 36
- no-connect marks 33 -> 35
Other:
- moved on the sheet: SH1
Changed lines of the file:
@@
 EESchema Schematic File Version 2
+LIBS:Aforino-rescue
 LIBS:power
 LIBS:device
 LIBS:switches
 LIBS:relays
-LIBS:motors
 LIBS:transistors
 LIBS:conn
@@
 LIBS:valves
 LIBS:ESP8266
-LIBS:myLib
-LIBS:Connector_Generic
-LIBS:Connector_Generic_Shielded
 LIBS:shield_arduino
 LIBS:dc-dc
+LIBS:Escolabs
+LIBS:myLib
 LIBS:Aforino-cache
 EELAYER 25 0
@@
 F 0 "Conn2" H 2600 4175 60  0000 C CNN
 F 1 "myConn3x1" H 2650 4575 60  0000 C CNN
-F 2 "myLib:myConn3x1" H 2650 4175 60  0001 C CNN
+F 2 "Escolabs:MyConn3x1" H 2650 4175 60  0001 C CNN
 F 3 "" H 2650 4175 60  0001 C CNN
 	1    2600 4375
@@
 F 0 "Conn1" H 2600 3375 60  0000 C CNN
 F 1 "myConn3x1" H 2650 3775 60  0000 C CNN
-F 2 "myLib:myConn3x1" H 2650 3375 60  0001 C CNN
+F 2 "Escolabs:MyConn3x1" H 2650 3375 60  0001 C CNN
 F 3 "" H 2650 3375 60  0001 C CNN
 	1    2600 3575
@@
 Text Label 3650 3575 0    60   ~ 0
 IR_IN
-Text Label 6525 2875 0    60   ~ 0
+Text Label 6575 2825 0    60   ~ 0
 IR_IN
 Text Label 3650 4375 0    60   ~ 0
 IR_OUT
-Text Label 6525 2775 0    60   ~ 0
+Text Label 6575 2700 0    60   ~ 0
 IR_OUT
-$Comp
-L SW_Push SW1
-U 1 1 5A627D48
-P 3300 6175
-F 0 "SW1" H 3350 6275 50  0000 L CNN
-F 1 "SW_Push" H 3300 6115 50  0000 C CNN
-F 2 "Buttons_Switches_THT:SW_PUSH_6mm" H 3300 6375 50  0001 C CNN
-F 3 "" H 3300 6375 50  0001 C CNN
-	1    3300 6175
-	1    0    0    -1
-$EndComp
-$Comp
-L ESP-Breatout-16Pin U1
-U 1 1 5A629AEC
-P 5300 5225
-F 0 "U1" H 5300 5125 50  0000 C CNN
-F 1 "ESP-Breatout-16Pin" H 5300 5625 50  0000 C CNN
-F 2 "myLib:ESP-Breakout-16PIN" H 5200 5225 50  0001 C CNN
-F 3 "" H 5200 5225 50  0001 C CNN
-	1    5300 5225
-	1    0    0    -1
-$EndComp
-$Comp
-L SW_Push SW2
-U 1 1 5A628F1B
-P 7500 5325
-F 0 "SW2" H 7550 5425 50  0000 L CNN
-F 1 "SW_Push" H 7500 5265 50  0000 C CNN
-F 2 "Buttons_Switches_THT:SW_PUSH_6mm" H 7500 5525 50  0001 C CNN
-F 3 "" H 7500 5525 50  0001 C CNN
-	1    7500 5325
-	1    0    0    -1
-$EndComp
 $Comp
 L GND #PWR08
@@
 $EndComp
 NoConn ~ 4300 5525
-NoConn ~ 4300 5425
-NoConn ~ 4300 5325
 NoConn ~ 4300 5225
 NoConn ~ 4300 5025
@@
 Text Label 6500 5125 0    60   ~ 0
 SCL
-Text Label 3700 6175 0    60   ~ 0
-FIRM_SW
 Text Label 6500 5425 0    60   ~ 0
 FIRM_SW
@@
 FIRM_SW
 $Comp
-L Conn_01x04_Female J1
+L Conn_01x04_Female-RESCUE-Aforino J1
 U 1 1 5A63E347
 P 8600 4625
@@
 	1    0    0    -1
 $EndComp
-$Comp
-L Conn_01x04_Female J2
-U 1 1 5A63E718
-P 6075 825
-F 0 "J2" H 6075 1025 50  0000 C CNN
-F 1 "Conn_01x04_Female" H 6075 525 50  0000 C CNN
-F 2 "Connector_PinHeader_2.54mm:PinHeader_1x04_P2.54mm_Vertical" H 6075 825 50  0001 C CNN
-F 3 "" H 6075 825 50  0001 C CNN
-	1    6075 825
-	1    0    0    -1
-$EndComp
-Text Label 5575 4125 3    60   ~ 0
+Text Label 5625 4175 3    60   ~ 0
 SDA
-Text Label 5425 4125 3    60   ~ 0
+Text Label 5500 4175 3    60   ~ 0
 SCL
-NoConn ~ 5875 725
 NoConn ~ 8400 4525
 $Comp
 L ARDUINO_MINI_PRO SH1
 U 1 1 5A63F347
-P 5325 2625
-F 0 "SH1" H 5325 2475 60  0000 C CNN
-F 1 "ARDUINO_MINI_PRO" H 5325 2625 60  0000 C CNN
-F 2 "SHIELD_ARDUINO:ARDUINO_MINI_PRO_V10" H 5150 4350 60  0001 C CNN
-F 3 "" H 5150 4350 60  0000 C CNN
-	1    5325 2625
-	1    0    0    -1
-$EndComp
-$Comp
-L GND #PWR09
-U 1 1 5A641268
-P 5875 1350
-F 0 "#PWR09" H 5875 1100 50  0001 C CNN
-F 1 "GND" H 5875 1200 50  0000 C CNN
-F 2 "" H 5875 1350 50  0001 C CNN
-F 3 "" H 5875 1350 50  0001 C CNN
-	1    5875 1350
-	1    0    0    -1
-$EndComp
-NoConn ~ 5225 3725
-NoConn ~ 5075 3725
-NoConn ~ 4525 3275
-NoConn ~ 4525 3175
-NoConn ~ 4525 3075
-NoConn ~ 4525 2975
-NoConn ~ 4525 2875
-NoConn ~ 4525 2775
-NoConn ~ 4525 2675
-NoConn ~ 4525 2575
-NoConn ~ 4525 2375
-NoConn ~ 4525 2275
-NoConn ~ 4525 2175
-NoConn ~ 6125 3275
-NoConn ~ 6125 3175
-NoConn ~ 6125 3075
-NoConn ~ 6125 2975
-NoConn ~ 6125 2675
-NoConn ~ 6125 2575
-NoConn ~ 6125 2375
-NoConn ~ 6125 2175
-NoConn ~ 5075 1425
-NoConn ~ 5625 1425
-$Comp
-L PWR_FLAG #FLG010
+P 5375 2675
+F 0 "SH1" H 5375 2525 60  0000 C CNN
+F 1 "ARDUINO_MINI_PRO" H 5375 2675 60  0000 C CNN
+F 2 "SHIELD_ARDUINO:ARDUINO_MINI_PRO_V10" H 5200 4400 60  0001 C CNN
+F 3 "" H 5200 4400 60  0000 C CNN
+	1    5375 2675
+	1    0    0    -1
+$EndComp
+NoConn ~ 5250 3775
+NoConn ~ 5125 3775
+NoConn ~ 5075 1500
+NoConn ~ 5700 1500
+$Comp
+L PWR_FLAG #FLG09
 U 1 1 5A62774C
 P 2950 2225
-F 0 "#FLG010" H 2950 2300 50  0001 C CNN
+F 0 "#FLG09" H 2950 2300 50  0001 C CNN
 F 1 "PWR_FLAG" H 2950 2375 50  0000 C CNN
 F 2 "" H 2950 2225 50  0001 C CNN
@@
 $EndComp
 $Comp
-L PWR_FLAG #FLG011
+L PWR_FLAG #FLG010
 U 1 1 5A627706
 P 2500 2225
-F 0 "#FLG011" H 2500 2300 50  0001 C CNN
+F 0 "#FLG010" H 2500 2300 50  0001 C CNN
 F 1 "PWR_FLAG" H 2500 2375 50  0000 C CNN
 F 2 "" H 2500 2225 50  0001 C CNN
@@
 $EndComp
 $Comp
-L GND #PWR012
+L GND #PWR011
 U 1 1 5A653773
 P 3900 1700
-F 0 "#PWR012" H 3900 1450 50  0001 C CNN
+F 0 "#PWR011" H 3900 1450 50  0001 C CNN
 F 1 "GND" H 3900 1550 50  0000 C CNN
 F 2 "" H 3900 1700 50  0001 C CNN
@@
 $EndComp
 $Comp
-L +3.3V #PWR013
+L +3.3V #PWR012
 U 1 1 5A65381F
 P 3900 1000
-F 0 "#PWR013" H 3900 850 50  0001 C CNN
+F 0 "#PWR012" H 3900 850 50  0001 C CNN
 F 1 "+3.3V" H 3900 1140 50  0000 C CNN
 F 2 "" H 3900 1000 50  0001 C CNN
@@
 	3000 3575 3650 3575
 Wire Wire Line
-	6125 2875 6525 2875
+	6175 2825 6575 2825
 Wire Wire Line
 	3000 4375 3650 4375
 Wire Wire Line
-	6125 2775 6525 2775
-Wire Wire Line
 	3000 4475 3250 4475
 Wire Wire Line
@@
 Wire Wire Line
 	3700 5125 4300 5125
-Wire Wire Line
-	7700 5325 7950 5325
 Wire Wire Line
 	6250 5525 7250 5525
@@
 Connection ~ 7250 5325
 Wire Wire Line
-	6250 5325 7300 5325
+	6250 5325 7550 5325
 Wire Wire Line
 	6250 5225 6500 5225
 Wire Wire Line
 	6250 5125 6500 5125
-Wire Wire Line
-	3100 6175 3100 5625
-Connection ~ 3100 5625
-Wire Wire Line
-	3500 6175 3750 6175
 Wire Wire Line
 	6250 5425 6500 5425
@@
 	7900 4825 8400 4825
 Wire Wire Line
-	5575 3725 5575 4125
-Wire Wire Line
-	5425 3725 5425 4125
-Wire Wire Line
-	5175 925  5875 925
-Wire Wire Line
-	5275 825  5875 825
-Wire Wire Line
-	5175 1425 5175 925
-Wire Wire Line
-	5275 1425 5275 825
+	5625 3775 5625 4175
+Wire Wire Line
+	5500 3775 5500 4175
 Wire Wire Line
 	2500 2225 2500 2375
@@
 	3550 1700 3900 1700
 Wire Wire Line
-	5525 1425 5525 1025
-NoConn ~ 6125 2275
+	3300 5925 3900 5925
+Text Label 3850 5925 0    60   ~ 0
+FIRM_SW
+Wire Wire Line
+	3200 5925 3200 5625
+Connection ~ 3200 5625
+$Comp
+L CONN_01X02 P1
+U 1 1 5AA28F0E
+P 3250 6125
+F 0 "P1" H 3250 6275 50  0000 C CNN
+F 1 "CONN_01X02" V 3350 6125 50  0000 C CNN
+F 2 "Pin_Headers:Pin_Header_Straight_1x02" H 3250 6125 50  0001 C CNN
+F 3 "" H 3250 6125 50  0000 C CNN
+	1    3250 6125
+	0    1    1    0
+$EndComp
+$Comp
+L CONN_01X02 P2
+U 1 1 5AA29366
+P 7600 5125
+F 0 "P2" H 7600 5275 50  0000 C CNN
+F 1 "CONN_01X02" V 7700 5125 50  0000 C CNN
+F 2 "Pin_Headers:Pin_Header_Straight_1x02" H 7600 5125 50  0001 C CNN
+F 3 "" H 7600 5125 50  0000 C CNN
+	1    7600 5125
+	0    -1   -1   0
+$EndComp
+Wire Wire Line
+	7650 5325 7950 5325
+$Comp
+L ESP-Breatout-16Pin U1
+U 1 1 5AA4641A
+P 5300 5225
+F 0 "U1" H 5300 5125 50  0000 C CNN
+F 1 "ESP-Breatout-16Pin" H 5300 5625 50  0000 C CNN
+F 2 "Escolabs:ESP8266-Breakout_Board-16Pin" H 5200 5225 50  0001 C CNN
+F 3 "" H 5200 5225 50  0001 C CNN
+	1    5300 5225
+	1    0    0    -1
+$EndComp
+NoConn ~ 6175 2075
+NoConn ~ 6175 2325
+NoConn ~ 6175 2450
+NoConn ~ 6175 2575
+NoConn ~ 6175 2950
+NoConn ~ 6175 3200
+NoConn ~ 6175 3325
+NoConn ~ 6175 3075
+Wire Wire Line
+	6575 2700 6175 2700
+NoConn ~ 6175 1950
+NoConn ~ 6175 2200
+NoConn ~ 4575 1950
+NoConn ~ 4575 2075
+NoConn ~ 4575 2200
+NoConn ~ 4575 2450
+NoConn ~ 4575 2575
+NoConn ~ 4575 2700
+NoConn ~ 4575 2825
+NoConn ~ 4575 2950
+NoConn ~ 4575 3075
+NoConn ~ 4575 3200
+NoConn ~ 4575 3325
+NoConn ~ 4295 5425
+NoConn ~ 4300 5325
+NoConn ~ 5325 1500
+NoConn ~ 5200 1500
+$Comp
+L GND #PWR013
+U 1 1 5AA48132
+P 5575 1350
+F 0 "#PWR013" H 5575 1100 50  0001 C CNN
+F 1 "GND" H 5575 1200 50  0000 C CNN
+F 2 "" H 5575 1350 50  0000 C CNN
+F 3 "" H 5575 1350 50  0000 C CNN
+	1    5575 1350
+	-1   0    0    1
+$EndComp
+Wire Wire Line
+	5575 1350 5575 1500
 $Comp
 L +3.3V #PWR014
-U 1 1 5A655BBC
-P 5425 1375
-F 0 "#PWR014" H 5425 1225 50  0001 C CNN
-F 1 "+3.3V" H 5425 1515 50  0000 C CNN
-F 2 "" H 5425 1375 50  0001 C CNN
-F 3 "" H 5425 1375 50  0001 C CNN
-	1    5425 1375
-	1    0    0    -1
-$EndComp
-Wire Wire Line
-	5425 1375 5425 1425
-Wire Wire Line
-	5525 1025 5875 1025
-Wire Wire Line
-	5525 1350 5875 1350
-Connection ~ 5525 1350
-NoConn ~ 6125 2475
-$Comp
-L GND #PWR015
-U 1 1 5A66689F
-P 4350 2475
-F 0 "#PWR015" H 4350 2225 50  0001 C CNN
-F 1 "GND" H 4350 2325 50  0000 C CNN
-F 2 "" H 4350 2475 50  0001 C CNN
-F 3 "" H 4350 2475 50  0001 C CNN
-	1    4350 2475
-	1    0    0    -1
-$EndComp
-Wire Wire Line
-	4525 2475 4350 2475
+U 1 1 5AA4830B
+P 5450 1150
+F 0 "#PWR014" H 5450 1000 50  0001 C CNN
+F 1 "+3.3V" H 5450 1290 50  0000 C CNN
+F 2 "" H 5450 1150 50  0000 C CNN
+F 3 "" H 5450 1150 50  0000 C CNN
+	1    5450 1150
+	1    0    0    -1
+$EndComp
+Wire Wire Line
+	5450 1500 5450 1150
+NoConn ~ 4575 2325
 $EndSCHEMATC
